Commit message: second commite

File: xingtian_sym_model/urdf/xingtian_sym_model.urdf (robot description, URDF)
Before this commit: robot xingtian_sym_model, 17 links, 16 joints
Joints:
- joint LF_hip_joint: origin xyz=0.20857 0.1825 -0.00081409 rpy=0 0 0 -> xyz=0.20857 0.1825 -0.00081409 rpy=0 -2.18 0
- joint LF_knee_joint: origin xyz=-0.0806 -0.016 -0.11447 rpy=0 0 0 -> xyz=-0.0806 -0.016 -0.11447 rpy=0 1.14 0
- joint LR_hip_joint: origin xyz=-0.20857 0.1825 -0.00081409 rpy=0 0 0 -> xyz=-0.20857 0.1825 -0.00081409 rpy=0 -2.18 0
- joint LR_knee_joint: origin xyz=0.0806 -0.016 -0.11447 rpy=0 0 0 -> xyz=0.0806 -0.016 -0.11447 rpy=0 1.14 0
- joint RF_hip_joint: origin xyz=0.20857 -0.1825 -0.00081409 rpy=0 0 0 -> xyz=0.20857 -0.1825 -0.00081409 rpy=0 -2.18 0
- joint RF_knee_joint: origin xyz=-0.0806 0.016 -0.11447 rpy=0 0 0 -> xyz=-0.0806 0.016 -0.11447 rpy=0 1.14 0
- joint RR_hip_joint: origin xyz=-0.20857 -0.1825 -0.00081409 rpy=0 0 0 -> xyz=-0.20857 -0.1825 -0.00081409 rpy=0 -2.18 0
- joint RR_knee_joint: origin xyz=0.0806 0.016 -0.11447 rpy=0 0 0 -> xyz=0.0806 0.016 -0.11447 rpy=0 1.14 0

Commit message: third commite

File: xingtian_sym_model/urdf/xingtian_sym_model.urdf (robot description, URDF)
Before this commit: robot xingtian_sym_model, 17 links, 16 joints
Links:
- link LF_hip: geometry collision mesh filename=../meshes/LF_hip.STL; visual mesh filename=../meshes/LF_hip.STL
- link LF_knee: geometry collision mesh filename=../meshes/LF_knee.STL; visual mesh filename=../meshes/LF_knee.STL
- link LF_wheel: geometry collision mesh filename=../meshes/LF_wheel.STL; visual mesh filename=../meshes/LF_wheel.STL
- link LR_hip: geometry collision mesh filename=../meshes/LR_hip.STL; visual mesh filename=../meshes/LR_hip.STL
- link LR_knee: geometry collision mesh filename=../meshes/LR_knee.STL; visual mesh filename=../meshes/LR_knee.STL
- link LR_wheel: geometry collision mesh filename=../meshes/LR_wheel.STL; visual mesh filename=../meshes/LR_wheel.STL
- link RF_hip: geometry collision mesh filename=../meshes/RF_hip.STL; visual mesh filename=../meshes/RF_hip.STL
- link RF_knee: geometry collision mesh filename=../meshes/RF_knee.STL; visual mesh filename=../meshes/RF_knee.STL
- link RF_wheel: geometry collision mesh filename=../meshes/RF_wheel.STL; visual mesh filename=../meshes/RF_wheel.STL
- link RR_hip: geometry collision mesh filename=../meshes/RR_hip.STL; visual mesh filename=../meshes/RR_hip.STL
- link RR_knee: geometry collision mesh filename=../meshes/RR_knee.STL; visual mesh filename=../meshes/RR_knee.STL
- link RR_wheel: geometry collision mesh filename=../meshes/RR_wheel.STL; visual mesh filename=../meshes/RR_wheel.STL
- link base_link: geometry collision mesh filename=../meshes/base_link.STL; visual mesh filename=../meshes/base_link.STL
- link imu_link: geometry collision mesh filename=../meshes/imu_link.STL; visual mesh filename=../meshes/imu_link.STL
Joints:
- joint LF_hip_joint: axis 0 1 0 -> 0 -1 0
- joint LF_knee_joint: axis 0 1 0 -> 0 -1 0
- joint LF_wheel_joint: axis 0 1 0 -> 0 -1 0; limit (none) -> lower=-6.28318 upper=6.28318 effort=10000 velocity=50; type continuous -> revolute
- joint LR_hip_joint: origin xyz=-0.20857 0.1825 -0.00081409 rpy=0 -2.18 0 -> xyz=-0.20857 0.1825 -0.00081409 rpy=0 2.18 0
- joint LR_knee_joint: origin xyz=0.0806 -0.016 -0.11447 rpy=0 1.14 0 -> xyz=0.0806 -0.016 -0.11447 rpy=0 -1.14 0
- joint LR_wheel_joint: limit (none) -> lower=-6.28318 upper=6.28318 effort=10000 velocity=50; type continuous -> revolute
- joint RF_wheel_joint: limit (none) -> lower=-6.28318 upper=6.28318 effort=10000 velocity=50; type continuous -> revolute
- joint RR_hip_joint: axis 0 -1 0 -> 0 1 0; origin xyz=-0.20857 -0.1825 -0.00081409 rpy=0 -2.18 0 -> xyz=-0.20857 -0.1825 -0.00081409 rpy=0 2.18 0
- joint RR_knee_joint: axis 0 -1 0 -> 0 1 0; origin xyz=0.0806 0.016 -0.11447 rpy=0 1.14 0 -> xyz=0.0806 0.016 -0.11447 rpy=0 -1.14 0
- joint RR_wheel_joint: axis 0 -1 0 -> 0 1 0; limit (none) -> lower=-6.28318 upper=6.28318 effort=10000 velocity=50; type continuous -> revolute

Commit message: fourth

File: xingtian_sym_model/urdf/xingtian_sym_model.urdf (robot description, URDF)
Before this commit: robot xingtian_sym_model, 17 links, 16 joints
Joints:
- joint LF_hip_joint: axis 0 -1 0 -> 0 1 0
- joint LF_knee_joint: axis 0 -1 0 -> 0 1 0
- joint LF_wheel_joint: axis 0 -1 0 -> 0 1 0
- joint LR_hip_joint: axis 0 1 0 -> 0 -1 0
- joint LR_knee_joint: axis 0 1 0 -> 0 -1 0
- joint LR_wheel_joint: axis 0 1 0 -> 0 -1 0
- joint RF_hip_joint: axis 0 -1 0 -> 0 1 0
- joint RF_knee_joint: axis 0 -1 0 -> 0 1 0
- joint RF_wheel_joint: axis 0 -1 0 -> 0 1 0
- joint RR_hip_joint: axis 0 1 0 -> 0 -1 0
- joint RR_knee_joint: axis 0 1 0 -> 0 -1 0
- joint RR_wheel_joint: axis 0 1 0 -> 0 -1 0

Commit message: fifth commit

File: xingtian_sym_model/urdf/xingtian_sym_model.urdf (robot description, URDF)
Before this commit: robot xingtian_sym_model, 17 links, 16 joints
Joints:
- joint LF_hip_joint: axis 0 1 0 -> 0 -1 0
- joint LF_knee_joint: axis 0 1 0 -> 0 -1 0
- joint LF_wheel_joint: axis 0 1 0 -> 0 -1 0
- joint LR_hip_joint: origin xyz=-0.20857 0.1825 -0.00081409 rpy=0 2.18 0 -> xyz=-0.20857 0.1825 -0.00081409 rpy=0 -2.18 0
- joint LR_knee_joint: origin xyz=0.0806 -0.016 -0.11447 rpy=0 -1.14 0 -> xyz=0.0806 -0.016 -0.11447 rpy=0 1.14 0
- joint RF_hip_joint: axis 0 1 0 -> 0 -1 0
- joint RF_knee_joint: axis 0 1 0 -> 0 -1 0
- joint RF_wheel_joint: axis 0 1 0 -> 0 -1 0
- joint RR_hip_joint: origin xyz=-0.20857 -0.1825 -0.00081409 rpy=0 2.18 0 -> xyz=-0.20857 -0.1825 -0.00081409 rpy=0 -2.18 0
- joint RR_knee_joint: origin xyz=0.0806 0.016 -0.11447 rpy=0 -1.14 0 -> xyz=0.0806 0.016 -0.11447 rpy=0 1.14 0
